File: 4_Fabrication/Version_00/C_KiCAD/Light_trainer/Light_trainer.sch (KiCad schematic (older format))
At the start: 21 parts

Commit message: modif kicad
Parts:
- removed C?: C, symbol Device:C
- removed D? (x2): LED, symbol Device:LED
- removed D? (x3): LED_BGRA, symbol Device:LED_BGRA
- removed J?: USB_B_Micro, symbol Connector:USB_B_Micro
- removed R? (x4): R, symbol Device:R
- removed SW? (x3): SW_Push, symbol Switch:SW_Push
- removed U?: ISL9301IRZ, symbol Battery_Management:ISL9301IRZ
- added C? (x3): C, symbol Device:C
- added D? (x7): LED, symbol Device:LED
- added D?: D, symbol Device:D
- added D?: D_Zener, symbol Device:D_Zener
- added D? (x3): LED_BGRA, symbol Device:LED_BGRA
- added J?: USB_B_Micro, symbol Connector:USB_B_Micro
- added Q?: Q_NJFET_DGS, symbol Device:Q_NJFET_DGS
- added R? (x19): R, symbol Device:R
- added SW? (x3): SW_Push, symbol Switch:SW_Push
- added U?: MCP73831-2-OT, Package_TO_SOT_SMD:SOT-23-5, symbol Battery_Management:MCP73831-2-OT
- added U? (x5): LM339, symbol Comparator:LM339
Connections:
- net labels added: +5V, aff, comm_LB, led_B, stat, switch
- wire segments 23 -> 125
Other:
- note added: "Affichage de la tension de la batterie"
- note added: "Charge de la batterie"
- note added: "Switch"
- moved on the sheet: R?, SW?

Commit message: modif kicad
Parts:
- removed J? (x2): Conn_01x15_Female, symbol Connector:Conn_01x15_Female
- added C? (x2): C, symbol Device:C
- added D?: ESDA6V1BC6, Package_TO_SOT_SMD:SOT-23-6, symbol Power_Protection:ESDA6V1BC6
- added D?: D_Schottky, symbol Device:D_Schottky
- added Q? (x2): S8050, Package_TO_SOT_THT:TO-92_Inline, symbol Transistor_BJT:S8050
- added R?: 2K, symbol Device:R
- added R?: 22.1K, symbol Device:R
- added R?: 47.5K, symbol Device:R
- added R? (x3): 10K, symbol Device:R
- added U?: ESP32-WROOM-32, RF_Module:ESP32-WROOM-32, symbol RF_Module:ESP32-WROOM-32
- added U?: LT1963AxST-3.3, Package_TO_SOT_SMD:SOT-223-3_TabPin2, symbol Regulator_Linear:LT1963AxST-3.3
- added U?: AP9101CK6, Package_TO_SOT_SMD:SOT-23-6, symbol Battery_Management:AP9101CK6
- added U?: CP2102N-A01-GQFN28, Package_DFN_QFN:QFN-28-1EP_5x5mm_P0.5mm_EP3.35x3.35mm, symbol Interface_USB:CP2102N-A01-GQFN28
Connections:
- net labels added: +3.3V, CTS, D+, D-, DCD, DSR, DTR, EN, IO0, RI, RTS, RXD, TXD
- wire segments 125 -> 189
- no-connect marks 0 -> 13
Other:
- note added: "Charge"
- note added: "Programmateur"
- note added: "Protect"
- note added: "régulateur 3.3v"
- note added: "stat de la charge"
- note added: "usb avec protect ESD"
- note removed: "Charge de la batterie"
- moved on the sheet: C?, D?, R?, SW?, U?

Commit message: modif kicad
add programateur, protection, esd
Parts:
- removed Q?: Q_NJFET_DGS, symbol Device:Q_NJFET_DGS
- added C? (x2): 10pF, symbol Device:C
- added C?: 100nF, symbol Device:C
- added C? (x2): 0,1uF, symbol Device:C
- added C?: 22uF, symbol Device:C
- added J?: Conn_charge_+, symbol Connector:Conn_01x01_Female
- added J?: Conn_charge_-, symbol Connector:Conn_01x01_Female
- added J?: Conn_Batt, symbol Connector:Conn_01x02_Female
- added Q? (x2): Q_DUAL_NMOS_DMN62D0UDW, symbol Device:Q_DUAL_NMOS_DMN62D0UDW
- added Q? (x3): 2N7002, Package_TO_SOT_SMD:SOT-23, symbol Transistor_FET:2N7002
- added R?: 330, symbol Device:R
- added R?: 2K7, symbol Device:R
- added R? (x6): R, symbol Device:R
- added R?: 10k, symbol Device:R
- added R? (x4): 10K, symbol Device:R
- added SW?: SW_DIP_x04, symbol Switch:SW_DIP_x04
- C?: value C -> 0,1uF
- C?: value C -> 4,7uF
- R?: value R -> 10k
Connections:
- net labels added: GND1, comm_LG, comm_LR, led_G, led_R
- wire segments 189 -> 288
Other:
- note added: "Auto program\nDTR RTS --> EN IO0\n 1 1 1 1\n 0 0 1 1\n 1 0 0 1\n 0 1 1 0"
- note added: "Charge et protection de la batterie"
- note added: "Driver Led"
- note added: "Led RGB"
- note added: "LightTrainer V00"
- note added: "Scélection master / slave"
- note added: "status de la charge"
- note removed: "stat de la charge"
- moved on the sheet: C?, D?, J?, Q?, R?, SW?, U?

Commit message: Modif kicad
Parts:
- removed C?: C, symbol Device:C
- removed D? (x5): LED, symbol Device:LED
- removed D?: D, symbol Device:D
- removed D?: D_Zener, symbol Device:D_Zener
- removed Q? (x3): 2N7002, Package_TO_SOT_SMD:SOT-23, symbol Transistor_FET:2N7002
- removed R? (x22): R, symbol Device:R
- removed SW?: SW_Push, symbol Switch:SW_Push
- removed U? (x5): LM339, symbol Comparator:LM339
- C? (x2): value C -> 4,7uF
- D?: value LED -> LED_R
- D?: value LED -> LED_G
- R? (x2): value R -> 470
- R?: value R -> 2K
Connections:
- net labels removed: -BATT, aff, comm_LB, comm_LG, comm_LR
- wire segments 288 -> 199
Other:
- note added: "LED_G - LED_R\n 1 - 0 -> Chargée\n 0 - 1 -> Charge\n 1 - 1 -> Error"
- note removed: "Affichage de la tension de la batterie"
- note removed: "Driver Led"
- moved on the sheet: C?, D?, J?, Q?, Q?A, Q?B, R?, SW?, U?

Commit message: add neo-pixel led
add néo-pixel led
add 3V to 5V
modif condo EN
add listes des composants
Parts:
- removed D? (x4): LED_BGRA, symbol Device:LED_BGRA
- added C?: 1uF, symbol Device:C
- added C?: 10uF, symbol Device:C
- added C? (x3): 10pF, symbol Device:C
- added D? (x10): SK6812, LED_SMD:LED_SK6812_PLCC4_5.0x5.0mm_P3.2mm, symbol LED:SK6812
- added L?: 10uH, Inductor_SMD:L_Wuerth_WE_PMI, symbol pspice:INDUCTOR
- added SW? (x2): SW_Push, symbol Switch:SW_Push
- added U?: LTC3525-5, Package_TO_SOT_SMD:SOT-363_SC-70-6, symbol Regulator_Switching:LTC3525-5
- C?: value 0,1uF -> 4,7uF
- J?: footprint (none) -> Connector_USB:USB_Micro-B_Wuerth_629105150521_CircularHoles; Fournisseur (none) -> Digikey; Prix total (none) -> 1.88; prix unité (none) -> 1,88
- J? (x2): footprint (none) -> Connector_Wire:SolderWire-0.1sqmm_1x01_D0.4mm_OD1mm
- J?: footprint (none) -> Connector_Wire:SolderWire-0.1sqmm_1x02_P3.6mm_D0.4mm_OD1mm_Relief
- R? (x15): footprint (none) -> Resistor_SMD:R_0805_2012Metric
- R?: value 22.1K -> 24K; footprint (none) -> Resistor_SMD:R_0805_2012Metric
- R?: value 47.5K -> 47K; footprint (none) -> Resistor_SMD:R_0805_2012Metric
- U?: Fournisseur (none) -> Digikey; Prix total (none) -> 0,51; prix unité (none) -> 0,51
- U?: Fournisseur (none) -> Digikey; Prix total (none) -> 3,82; prix unité (none) -> 3,82
- U?: Fournisseur (none) -> Digikey; Prix total (none) -> 5; prix unité (none) -> 5
- U?: Fournisseur (none) -> Digikey; Prix total (none) -> 0,4; prix unité (none) -> 0,4
- U?: Fournisseur (none) -> Digikey; Prix total (none) -> 2,88; prix unité (none) -> 2,88
Connections:
- net labels added: +5VA, DOUT, LED
- net labels removed: led_B, led_G, led_R
- wire segments 199 -> 227
- no-connect marks 13 -> 14
Other:
- note added: "3V - 4.2V to 5V"
- note added: "LED néo-pixel"
- note added: "USB to UART"
- note removed: "Led RGB"
- note removed: "Programmateur"
- moved on the sheet: C?, U?

Commit message: modif Kicad
Parts:
- removed C?: 10pF, symbol Device:C
Changed lines of the file:
@@
 Text Notes 5200 7250 0    50   ~ 0
 LED néo-pixel
-$Comp
-L Device:C C?
-U 1 1 60165D5E
-P 6300 7500
-F 0 "C?" H 6415 7546 50  0000 L CNN
-F 1 "10pF" H 6415 7455 50  0000 L CNN
-F 2 "" H 6338 7350 50  0001 C CNN
-F 3 "~" H 6300 7500 50  0001 C CNN
-	1    6300 7500
-	0    -1   -1   0
-$EndComp
 $EndSCHEMATC

Commit message: add label
Parts:
- added R? (x2): R, symbol Device:R
- C? (x2): value 10pF -> 0,1uF
- Q? (x2): symbol Device:Q_DUAL_NMOS_DMN62D0UDW -> Light_trainer-rescue:Q_DUAL_NMOS_DMN62D0UDW-Device
Connections:
- net +BATT: now also R?.1
- net EN: now also C?.1, SW?.2
- net GND: now also C?.2, C?.2, SW?.1, SW?.1, R?.2
- net IO0: now also C?.1, SW?.2
- new net: R?.1, R?.2
Other:
- moved on the sheet: C?
Changed lines of the file:
@@
 Rev ""
 Comp ""
-Comment1 "©Robin Forestier 2020/2021"
+Comment1 "©2021 Robin Forestier"
 Comment2 ""
 Comment3 "V_00"
@@
 Wire Notes Line
 	3400 7450 3400 9850
-Text Notes 3400 7350 0    50   ~ 0
+Text Notes 3400 7400 0    50   ~ 0
 Switch
 $Comp
@@
 	2400 4700 2400 4950
 $Comp
-L Device:Q_DUAL_NMOS_DMN62D0UDW Q?
+L Light_trainer-rescue:Q_DUAL_NMOS_DMN62D0UDW-Device Q?
 U 1 1 5FF8AF5B
 P 2950 5700
@@
 $EndComp
 $Comp
-L Device:Q_DUAL_NMOS_DMN62D0UDW Q?
+L Light_trainer-rescue:Q_DUAL_NMOS_DMN62D0UDW-Device Q?
 U 2 1 5FF8BD1C
 P 3450 5700
@@
 U 1 1 600FA458
 P 10550 6200
-F 0 "SW?" H 10550 6485 50  0000 C CNN
-F 1 "SW_Push" H 10550 6394 50  0000 C CNN
+F 0 "SW?" H 10550 6450 50  0000 C CNN
+F 1 "SW_Push" H 10550 6350 50  0000 C CNN
 F 2 "" H 10550 6400 50  0001 C CNN
 F 3 "~" H 10550 6400 50  0001 C CNN
@@
 U 1 1 60108309
 P 10550 6850
-F 0 "SW?" H 10550 7135 50  0000 C CNN
-F 1 "SW_Push" H 10550 7044 50  0000 C CNN
+F 0 "SW?" H 10550 7100 50  0000 C CNN
+F 1 "SW_Push" H 10550 7000 50  0000 C CNN
 F 2 "" H 10550 7050 50  0001 C CNN
 F 3 "~" H 10550 7050 50  0001 C CNN
@@
 L Device:C C?
 U 1 1 60116593
-P 10850 6400
-F 0 "C?" H 10965 6446 50  0000 L CNN
-F 1 "10pF" H 10965 6355 50  0000 L CNN
-F 2 "" H 10888 6250 50  0001 C CNN
-F 3 "~" H 10850 6400 50  0001 C CNN
-	1    10850 6400
-	1    0    0    -1
+P 10550 6350
+F 0 "C?" V 10600 6400 50  0000 L CNN
+F 1 "0,1uF" V 10700 6400 50  0000 L CNN
+F 2 "" H 10588 6200 50  0001 C CNN
+F 3 "~" H 10550 6350 50  0001 C CNN
+	1    10550 6350
+	0    1    1    0
 $EndComp
 $Comp
 L Device:C C?
 U 1 1 601244B2
-P 10850 7050
-F 0 "C?" H 10965 7096 50  0000 L CNN
-F 1 "10pF" H 10965 7005 50  0000 L CNN
-F 2 "" H 10888 6900 50  0001 C CNN
-F 3 "~" H 10850 7050 50  0001 C CNN
-	1    10850 7050
-	1    0    0    -1
+P 10550 7050
+F 0 "C?" V 10600 7100 50  0000 L CNN
+F 1 "0,1uF" V 10700 7100 50  0000 L CNN
+F 2 "" H 10588 6900 50  0001 C CNN
+F 3 "~" H 10550 7050 50  0001 C CNN
+	1    10550 7050
+	0    1    1    0
 $EndComp
 Text GLabel 5600 8000 0    50   Input ~ 0
@@
 Text Notes 5200 7250 0    50   ~ 0
 LED néo-pixel
+$Comp
+L power:+BATT #PWR?
+U 1 1 5FDF6111
+P 13950 2450
+F 0 "#PWR?" H 13950 2300 50  0001 C CNN
+F 1 "+BATT" H 13965 2623 50  0000 C CNN
+F 2 "" H 13950 2450 50  0001 C CNN
+F 3 "" H 13950 2450 50  0001 C CNN
+	1    13950 2450
+	1    0    0    -1
+$EndComp
+Wire Wire Line
+	13950 2450 13950 2500
+$Comp
+L Device:R R?
+U 1 1 5FE04B03
+P 13950 2650
+F 0 "R?" H 14020 2696 50  0000 L CNN
+F 1 "R" H 14020 2605 50  0000 L CNN
+F 2 "" V 13880 2650 50  0001 C CNN
+F 3 "~" H 13950 2650 50  0001 C CNN
+	1    13950 2650
+	1    0    0    -1
+$EndComp
+$Comp
+L Device:R R?
+U 1 1 5FE054D4
+P 13950 3050
+F 0 "R?" H 14020 3096 50  0000 L CNN
+F 1 "R" H 14020 3005 50  0000 L CNN
+F 2 "" V 13880 3050 50  0001 C CNN
+F 3 "~" H 13950 3050 50  0001 C CNN
+	1    13950 3050
+	1    0    0    -1
+$EndComp
+Wire Wire Line
+	13950 2800 13950 2850
+Wire Wire Line
+	13950 3200 13950 3250
+$Comp
+L power:GND #PWR?
+U 1 1 5FE3132C
+P 13950 3250
+F 0 "#PWR?" H 13950 3000 50  0001 C CNN
+F 1 "GND" H 13955 3077 50  0000 C CNN
+F 2 "" H 13950 3250 50  0001 C CNN
+F 3 "" H 13950 3250 50  0001 C CNN
+	1    13950 3250
+	1    0    0    -1
+$EndComp
+Wire Wire Line
+	13950 2850 13800 2850
+Connection ~ 13950 2850
+Wire Wire Line
+	13950 2850 13950 2900
+Text GLabel 13050 2700 2    50   Output ~ 0
+LED
+Wire Wire Line
+	10400 6350 10300 6350
+Wire Wire Line
+	10300 6350 10300 6200
+Wire Wire Line
+	10300 6200 10350 6200
+Wire Wire Line
+	10400 7050 10300 7050
+Wire Wire Line
+	10300 7050 10300 6850
+Wire Wire Line
+	10300 6850 10350 6850
+$Comp
+L power:GND #PWR?
+U 1 1 5FE9C565
+P 10300 7150
+F 0 "#PWR?" H 10300 6900 50  0001 C CNN
+F 1 "GND" H 10200 7150 50  0000 C CNN
+F 2 "" H 10300 7150 50  0001 C CNN
+F 3 "" H 10300 7150 50  0001 C CNN
+	1    10300 7150
+	1    0    0    -1
+$EndComp
+Wire Wire Line
+	10300 7150 10300 7050
+Connection ~ 10300 7050
+$Comp
+L power:GND #PWR?
+U 1 1 5FEE889C
+P 10300 6450
+F 0 "#PWR?" H 10300 6200 50  0001 C CNN
+F 1 "GND" H 10200 6450 50  0000 C CNN
+F 2 "" H 10300 6450 50  0001 C CNN
+F 3 "" H 10300 6450 50  0001 C CNN
+	1    10300 6450
+	1    0    0    -1
+$EndComp
+Wire Wire Line
+	10300 6450 10300 6350
+Connection ~ 10300 6350
+Wire Wire Line
+	10700 6350 10800 6350
+Wire Wire Line
+	10800 6350 10800 6200
+Wire Wire Line
+	10800 6200 10750 6200
+Wire Wire Line
+	10700 7050 10800 7050
+Wire Wire Line
+	10800 7050 10800 6850
+Wire Wire Line
+	10800 6850 10750 6850
+Text GLabel 11050 6200 2    50   Output ~ 0
+IO0
+Wire Wire Line
+	11050 6200 10800 6200
+Connection ~ 10800 6200
+Text GLabel 11050 6850 2    50   Output ~ 0
+EN
+Wire Wire Line
+	11050 6850 10800 6850
+Connection ~ 10800 6850
 $EndSCHEMATC
