File: 4_Fabrication/Version_00/C_KiCAD/Light_trainer/Light_trainer.sch (KiCad schematic (older format))
At the start: 61 parts

Commit message: modif kicad
Parts:
- added C14: 10uF, Capacitor_SMD:C_0805_2012Metric, symbol Device:C
- added C15: 0,1uF, Capacitor_SMD:C_0805_2012Metric, symbol Device:C
- added D10: LED_R, LED_SMD:LED_1806_4516Metric, symbol Device:LED
- added D11, D12, D13: LED_G, LED_SMD:LED_1806_4516Metric, symbol Device:LED
- added R12: 68R, Resistor_SMD:R_0805_2012Metric, symbol Device:R
- added R9: 10K, Resistor_SMD:R_0805_2012Metric, symbol Device:R
- added S1: SW_DP3T, Button_Switch_THT:SW_DP3T, symbol Switch:SW_DP3T
- added TP1, TP2, TP3, TP4: TestPoint, TestPoint:TestPoint_THTPad_2.5x2.5mm_Drill1.2mm, symbol Connector:TestPoint
- R2: renamed from R?; value 470 -> 150
- R3: renamed from R?; value 40k -> 4k
- R4: renamed from R?; value 470 -> 100
- R5: renamed from R?; value 100k -> 10k
- gave numbers to parts that had none: 57
Connections:
- net labels added: LED_B_0, LED_B_1, LED_B_2, LED_B_3, batt_on, info_batt
- wire segments 242 -> 290
- no-connect marks 15 -> 33
Other:
- note added: "Affichage tension de la batteire"
- note added: "ESP 32"
- note added: "R G G G Batterie\n1 1 1 1 => 100%\n1 1 1 0 => 75%\n1 1 0 0 => 50%\n1 0 0 0 => 25%"
- note added: "interupteur principal + affichage batterie"
- moved on the sheet: C10, C11, C12, C13, C3, C5, C6, C7, C8, C9, D1, D14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

Commit message: modif kicad
first layout
8 néo pixel
Parts:
- removed D18, D9: SK6812, LED_SMD:LED_SK6812_PLCC4_5.0x5.0mm_P3.2mm, symbol LED:SK6812
- Q2, Q3: footprint Package_TO_SOT_THT:TO-92_Inline -> Package_TO_SOT_SMD:SOT-23
- renumbered D11 to D10, D12 to D11, D13 to D12, D14 to D13, D15 to D14, D16 to D15, D17 to D16, D10 to D9
Connections:
- wire segments 290 -> 284
Other:
- moved on the sheet: TP5

Commit message: modif kicad
Parts:
- removed Q1: DMG3414U, Package_TO_SOT_SMD:SOT-23, symbol Transistor_FET:DMG3414U
- removed R7: 100k, Resistor_SMD:R_0805_2012Metric, symbol Device:R
- added J3, J4: Conn_01x09_Female, Connector_PinHeader_1.00mm:PinHeader_1x09_P1.00mm_Vertical, symbol Connector:Conn_01x09_Female
- C9: value 10uF -> 1uF
Connections:
- wire segments 284 -> 294
Other:
- moved on the sheet: C8, C9, J2, R8, U4

Commit message: modif kicad
Parts:
- added J5: Conn_01x02_Batterie, Connector_Wire:SolderWire-0.1sqmm_1x02_P3.6mm_D0.4mm_OD1mm, symbol Connector:Conn_01x02_Female
Connections:
- net GND: now also J5.1 (Pin_1)
- net VBUS: now also J5.2 (Pin_2)
Other:
- moved on the sheet: J2
Changed lines of the file:
@@
 L Connector:Conn_01x02_Female J2
 U 1 1 6012C36F
-P 4150 4850
-F 0 "J2" H 4150 4600 50  0000 L CNN
-F 1 "Conn_01x02_Batterie" H 3600 4350 50  0000 L CNN
-F 2 "Connector_JST:JST_PH_B2B-PH-K_1x02_P2.00mm_Vertical" H 4150 4850 50  0001 C CNN
-F 3 "~" H 4150 4850 50  0001 C CNN
-	1    4150 4850
+P 4200 5150
+F 0 "J2" H 4200 4900 50  0000 L CNN
+F 1 "Conn_01x02_Batterie" H 3650 4700 50  0000 L CNN
+F 2 "Connector_JST:JST_PH_B2B-PH-K_1x02_P2.00mm_Vertical" H 4200 5150 50  0001 C CNN
+F 3 "~" H 4200 5150 50  0001 C CNN
+	1    4200 5150
 	-1   0    0    1
 $EndComp
@@
 L power:GND #PWR026
 U 1 1 60157F02
-P 4450 4950
-F 0 "#PWR026" H 4450 4700 50  0001 C CNN
-F 1 "GND" H 4455 4777 50  0000 C CNN
-F 2 "" H 4450 4950 50  0001 C CNN
-F 3 "" H 4450 4950 50  0001 C CNN
-	1    4450 4950
-	1    0    0    -1
-$EndComp
-Wire Wire Line
-	4450 4950 4450 4850
-Wire Wire Line
-	4350 4850 4450 4850
-Wire Wire Line
-	4350 4750 4450 4750
-Wire Wire Line
-	4450 4650 4450 4750
+P 4500 5250
+F 0 "#PWR026" H 4500 5000 50  0001 C CNN
+F 1 "GND" H 4505 5077 50  0000 C CNN
+F 2 "" H 4500 5250 50  0001 C CNN
+F 3 "" H 4500 5250 50  0001 C CNN
+	1    4500 5250
+	1    0    0    -1
+$EndComp
+Wire Wire Line
+	4500 5250 4500 5150
+Wire Wire Line
+	4400 5150 4500 5150
+Wire Wire Line
+	4400 5050 4500 5050
+Wire Wire Line
+	4500 4950 4500 5050
 $Comp
 L power:+BATT #PWR023
 U 1 1 601D8136
-P 4450 4650
-F 0 "#PWR023" H 4450 4500 50  0001 C CNN
-F 1 "+BATT" H 4465 4823 50  0000 C CNN
-F 2 "" H 4450 4650 50  0001 C CNN
-F 3 "" H 4450 4650 50  0001 C CNN
-	1    4450 4650
+P 4500 4950
+F 0 "#PWR023" H 4500 4800 50  0001 C CNN
+F 1 "+BATT" H 4515 5123 50  0000 C CNN
+F 2 "" H 4500 4950 50  0001 C CNN
+F 3 "" H 4500 4950 50  0001 C CNN
+	1    4500 4950
 	1    0    0    -1
 $EndComp
@@
 Wire Notes Line
 	3100 7600 5100 7600
+$Comp
+L Connector:Conn_01x02_Female J5
+U 1 1 5FFDC6C0
+P 4200 4300
+F 0 "J5" H 4200 4050 50  0000 L CNN
+F 1 "Conn_01x02_Batterie" H 3700 3850 50  0000 L CNN
+F 2 "Connector_Wire:SolderWire-0.1sqmm_1x02_P3.6mm_D0.4mm_OD1mm" H 4200 4300 50  0001 C CNN
+F 3 "~" H 4200 4300 50  0001 C CNN
+	1    4200 4300
+	-1   0    0    1
+$EndComp
+$Comp
+L power:GND #PWR067
+U 1 1 5FFF5AA7
+P 4500 4400
+F 0 "#PWR067" H 4500 4150 50  0001 C CNN
+F 1 "GND" H 4505 4227 50  0000 C CNN
+F 2 "" H 4500 4400 50  0001 C CNN
+F 3 "" H 4500 4400 50  0001 C CNN
+	1    4500 4400
+	1    0    0    -1
+$EndComp
+Wire Wire Line
+	4500 4400 4500 4300
+Wire Wire Line
+	4400 4300 4500 4300
+Wire Wire Line
+	4400 4200 4500 4200
+Wire Wire Line
+	4500 4100 4500 4200
+$Comp
+L power:VBUS #PWR066
+U 1 1 6004320F
+P 4500 4100
+F 0 "#PWR066" H 4500 3950 50  0001 C CNN
+F 1 "VBUS" H 4515 4273 50  0000 C CNN
+F 2 "" H 4500 4100 50  0001 C CNN
+F 3 "" H 4500 4100 50  0001 C CNN
+	1    4500 4100
+	1    0    0    -1
+$EndComp
 $EndSCHEMATC

Commit message: add datasheet
Restart the project
Parts:
- removed C1: 22uF, Capacitor_SMD:C_0805_2012Metric, symbol Device:C
- removed C10, C14, C3, C5, C7, C8: 10uF, Capacitor_SMD:C_0805_2012Metric, symbol Device:C
- removed C11, C13, C15, C2: 0,1uF, Capacitor_SMD:C_0805_2012Metric, symbol Device:C
- removed C12, C6, C9: 1uF, Capacitor_SMD:C_0805_2012Metric, symbol Device:C
- removed C4: 4,7uF, Capacitor_SMD:C_0805_2012Metric, symbol Device:C
- removed D1, D9: LED_R, LED_SMD:LED_1806_4516Metric, symbol Device:LED
- removed D10, D11, D12, D3: LED_G, LED_SMD:LED_1806_4516Metric, symbol Device:LED
- removed D2: ESDA6V1BC6, Package_TO_SOT_SMD:SOT-23-6, symbol Power_Protection:ESDA6V1BC6
- removed D4: MBR0540, Diode_SMD:D_SOD-123, symbol Diode:MBR0540
- removed J1: USB_B_Micro, Connector_USB:USB_Micro-B_Wuerth_629105150521_CircularHoles, symbol Connector:USB_B_Micro
- removed J2: Conn_01x02_Batterie, Connector_JST:JST_PH_B2B-PH-K_1x02_P2.00mm_Vertical, symbol Connector:Conn_01x02_Female
- removed J3, J4: Conn_01x09_Female, Connector_PinHeader_1.00mm:PinHeader_1x09_P1.00mm_Vertical, symbol Connector:Conn_01x09_Female
- removed J5: Conn_01x02_Batterie, Connector_Wire:SolderWire-0.1sqmm_1x02_P3.6mm_D0.4mm_OD1mm, symbol Connector:Conn_01x02_Female
- removed L1: 10uH, Inductor_SMD:L_Wuerth_WE_PMI, symbol pspice:INDUCTOR
- removed Q2, Q3: S8050, Package_TO_SOT_SMD:SOT-23, symbol Transistor_BJT:S8050
- removed R1, R5, R8: 10k, Resistor_SMD:R_0805_2012Metric, symbol Device:R
- removed R10, R11, R13, R14, R15, R16, R9: 10K, Resistor_SMD:R_0805_2012Metric, symbol Device:R
- removed R12: 68R, Resistor_SMD:R_0805_2012Metric, symbol Device:R
- removed R2: 150, Resistor_SMD:R_0805_2012Metric, symbol Device:R
- removed R3: 4k, Resistor_SMD:R_0805_2012Metric, symbol Device:R
- removed R4: 100, Resistor_SMD:R_0805_2012Metric, symbol Device:R
- removed R6: 2K, Resistor_SMD:R_0805_2012Metric, symbol Device:R
- removed S1: SW_DP3T, Button_Switch_THT:SW_DP3T, symbol Switch:SW_DP3T
- removed SW1, SW2: SW_Push, Button_Switch_SMD:SW_SPST_PTS645, symbol Switch:SW_Push
- removed SW6: SW_DIP_x04, Package_DIP:SMDIP-8_W7.62mm, symbol Switch:SW_DIP_x04
- removed TP1, TP2: TestPoint, TestPoint:TestPoint_THTPad_2.5x2.5mm_Drill1.2mm, symbol Connector:TestPoint
- removed U1: MCP73831-2-OT, Package_TO_SOT_SMD:SOT-23-5, symbol Battery_Management:MCP73831-2-OT
- removed U2: ESP32-WROOM-32, RF_Module:ESP32-WROOM-32, symbol RF_Module:ESP32-WROOM-32
- removed U3: LTC3525-5, Package_TO_SOT_SMD:SOT-363_SC-70-6, symbol Regulator_Switching:LTC3525-5
- removed U4: AP2112K-3.3, Package_TO_SOT_SMD:SOT-23-5, symbol Regulator_Linear:AP2112K-3.3
- removed U5: CP2104, Package_DFN_QFN:QFN-24-1EP_4x4mm_P0.5mm_EP2.6x2.6mm, symbol Interface_USB:CP2104
- added BT?: Battery, symbol Device:Battery
- added U1: ESP32-DevKitC-32D, Work_Forestier:ESP32-DevKitC-32D, symbol Work_Forestier:ESP32-DevKitC-32D
- D13, D14, D15, D16, D5, D6, D7, D8: symbol LED:SK6812 -> Light_trainer-rescue:SK6812-LED
- R17: symbol Device:R -> Light_trainer-rescue:R-Device
- SW3, SW4, SW5, SW7: symbol Switch:SW_Push -> Light_trainer-rescue:SW_Push-Switch
- TP3, TP4, TP5: symbol Connector:TestPoint -> Light_trainer-rescue:TestPoint-Connector
Connections:
- no-connect marks 33 -> 0
Other:
- note removed: "3V - 4.2V to 5V"
- note removed: "Affichage tension de la batteire"
- note removed: "Auto program\n\nDTR RTS --> EN IO0\n 1 1 1 1\n 0 0 1 1\n 1 0 0 1\n 0 1 1 0"
- note removed: "Charge"
- note removed: "Charge et protection de la batterie"
- note removed: "ESP 32"
- note removed: "LED_G - LED_R\n 1 - 0 -> Chargée\n 0 - 1 -> Charge\n 1 - 1 -> Error"
- note removed: "R G G G Batterie\n1 1 1 1 => 100%\n1 1 1 0 => 75%\n1 1 0 0 => 50%\n1 0 0 0 => 25%"
- note removed: "Scélection master / slave"
- note removed: "Si Vbatt = 4.2V \nIO2 = 3V\n30 uA"
- note removed: "USB to UART"
- note removed: "interupteur principal + affichage batterie"
- note removed: "status de la charge"
- note removed: "usb avec protect ESD"
- moved on the sheet: D13, D14, D15, D16, D5, D6, D7, D8, R17, SW3, SW4, SW5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

Commit message: add footprint
Parts:
- removed D13, D14, D15: SK6812, LED_SMD:LED_SK6812_PLCC4_5.0x5.0mm_P3.2mm, symbol Light_trainer-rescue:SK6812-LED
- added C1: 1uF, Capacitor_SMD:C_0805_2012Metric, symbol Device:C
- added C2: 10uF, Capacitor_SMD:C_0805_2012Metric, symbol Device:C
- added JP1: Jumper, Jumper:SolderJumper-2_P1.3mm_Open_Pad1.0x1.5mm, symbol Device:Jumper
- added L1: 10uH, Inductor_SMD:L_1210_3225Metric, symbol Device:L
- added TP2, TP3, TP6, TP7, TP8: TestPoint, TestPoint:TestPoint_THTPad_2.5x2.5mm_Drill1.2mm, symbol Connector:TestPoint
- added U1: LTC3525-5, Package_TO_SOT_SMD:SOT-363_SC-70-6, symbol Regulator_Switching:LTC3525-5
- R1: renamed from R17; footprint Resistor_SMD:R_0805_2012Metric -> Resistor_SMD:R_1206_3216Metric
- SW1: renamed from SW3; footprint Button_Switch_SMD:SW_SPST_PTS645 -> (none)
- SW2: renamed from SW4; footprint Button_Switch_SMD:SW_SPST_PTS645 -> (none)
- SW3: renamed from SW5; footprint Button_Switch_SMD:SW_SPST_PTS645 -> (none)
- SW4: renamed from SW7; footprint Button_Switch_SMD:SW_SPST_PTS645 -> (none)
- gave numbers to parts that had none: 1
- renumbered D5 to D1, D6 to D2, D7 to D3, D8 to D4, D16 to D5, TP4 to TP1, TP3 to TP4, U1 to U2
Connections:
- net DOUT is gone; now on an unnamed net: D4.4 (DOUT)
- net +3V3: now also U2.3V3, TP8.1
- net +5V: now also U2.5V, C2.1, TP7.1, U1.4 (VOUT)
- net GND: now also BT1.2 (-), U2.GND0, U2.GND1, U2.GND2, C1.2, C2.2, TP3.1, TP6.1, U1.2 (GND), U1.5 (GND)
- net LED: now also U2.IO16
- net switch: now also U2.IO17
- net at BT1.1 (+): now also JP1.1
- new net: C1.1, JP1.2, L1.1, TP2.1, U1.1 (~SHDN), U1.3 (VIN)
- new net: L1.2, U1.6 (SW)
- no-connect marks 0 -> 31
Other:
- note added: "Alimentation 3 pile AA avec régulateur 5V\n"
- note added: "ESP DEVKIT C\n"
- note added: "Test point GND/5V\n"
- moved on the sheet: BT1, D1, D2, D3, D4, D5, R1, SW1, SW2, SW3, SW4, TP1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

Commit message: ADD all footprint
All footprint
miss 1 3d (battery holder 3xAA)
Parts:
- BT1: footprint (none) -> Battery:BatteryHolder_TruPower_BH-331P_3xAA
- SW1, SW2, SW3, SW4: footprint (none) -> Work_Forestier:SW_Cherry_MX_1.00u_PCB_3D
Changed lines of the file:
@@
 F 0 "SW1" H 1600 4285 50  0000 C CNN
 F 1 "SW_Push" H 1600 4194 50  0000 C CNN
-F 2 "" H 1600 4200 50  0001 C CNN
+F 2 "Work_Forestier:SW_Cherry_MX_1.00u_PCB_3D" H 1600 4200 50  0001 C CNN
 F 3 "https://www.ckswitches.com/media/1471/pts645.pdf" H 1600 4200 50  0001 C CNN
 F 4 "Digikey" H 1600 4000 50  0001 C CNN "Fournisseur"
@@
 F 0 "SW2" H 1600 4635 50  0000 C CNN
 F 1 "SW_Push" H 1600 4544 50  0000 C CNN
-F 2 "" H 1600 4550 50  0001 C CNN
+F 2 "Work_Forestier:SW_Cherry_MX_1.00u_PCB_3D" H 1600 4550 50  0001 C CNN
 F 3 "https://www.ckswitches.com/media/1471/pts645.pdf" H 1600 4550 50  0001 C CNN
 F 4 "Digikey" H 1600 4350 50  0001 C CNN "Fournisseur"
@@
 F 0 "SW3" H 1600 4985 50  0000 C CNN
 F 1 "SW_Push" H 1600 4894 50  0000 C CNN
-F 2 "" H 1600 4900 50  0001 C CNN
+F 2 "Work_Forestier:SW_Cherry_MX_1.00u_PCB_3D" H 1600 4900 50  0001 C CNN
 F 3 "https://www.ckswitches.com/media/1471/pts645.pdf" H 1600 4900 50  0001 C CNN
 F 4 "Digikey" H 1600 4700 50  0001 C CNN "Fournisseur"
@@
 F 0 "SW4" H 1600 5335 50  0000 C CNN
 F 1 "SW_Push" H 1600 5244 50  0000 C CNN
-F 2 "" H 1600 5250 50  0001 C CNN
+F 2 "Work_Forestier:SW_Cherry_MX_1.00u_PCB_3D" H 1600 5250 50  0001 C CNN
 F 3 "https://www.ckswitches.com/media/1471/pts645.pdf" H 1600 5250 50  0001 C CNN
 F 4 "Digikey" H 1600 5050 50  0001 C CNN "Fournisseur"
@@
 F 0 "BT1" H 1308 2446 50  0000 L CNN
 F 1 "Battery" H 1308 2355 50  0000 L CNN
-F 2 "" V 1200 2460 50  0001 C CNN
+F 2 "Battery:BatteryHolder_TruPower_BH-331P_3xAA" V 1200 2460 50  0001 C CNN
 F 3 "~" V 1200 2460 50  0001 C CNN
 	1    1200 2400

Commit message: add all 3D
Parts:
- BT1: footprint Battery:BatteryHolder_TruPower_BH-331P_3xAA -> Work_Forestier:BatteryHolder_Keystone_2464_3xAA
Changed lines of the file:
@@
 F 0 "BT1" H 1308 2446 50  0000 L CNN
 F 1 "Battery" H 1308 2355 50  0000 L CNN
-F 2 "Battery:BatteryHolder_TruPower_BH-331P_3xAA" V 1200 2460 50  0001 C CNN
+F 2 "Work_Forestier:BatteryHolder_Keystone_2464_3xAA" V 1200 2460 50  0001 C CNN
 F 3 "~" V 1200 2460 50  0001 C CNN
 	1    1200 2400
