File: 4_Fabrication/Version_00/C_KiCAD/Light_trainer/Light_trainer.sch (KiCad schematic (older format))
At the start: 25 parts, among them SW1 SW_Push, SW2 SW_Push, SW3 SW_Push, SW4 SW_Push, U1 LTC3525-5, U2 ESP32-DevKitC-32D

Commit message: placement + routage
Parts:
- added SW5: SW_SPDT, Work_Forestier:C&K-1101M2S5CQE2, symbol Switch:SW_SPDT
Connections:
- net at BT1.1 (+): now also SW5.2 (B); no longer JP1.1
- new net: JP1.1, SW5.1 (A)
- no-connect marks 31 -> 32
Other:
- moved on the sheet: BT1, C1, C2, JP1, L1, TP2, TP3, U1
Changed lines of the file:
@@
 L Device:Battery BT1
 U 1 1 613C716D
-P 1200 2400
-F 0 "BT1" H 1308 2446 50  0000 L CNN
-F 1 "Battery" H 1308 2355 50  0000 L CNN
-F 2 "Work_Forestier:BatteryHolder_Keystone_2464_3xAA" V 1200 2460 50  0001 C CNN
-F 3 "~" V 1200 2460 50  0001 C CNN
-	1    1200 2400
+P 1000 2450
+F 0 "BT1" H 1108 2496 50  0000 L CNN
+F 1 "Battery" H 1108 2405 50  0000 L CNN
+F 2 "Work_Forestier:BatteryHolder_Keystone_2464_3xAA" V 1000 2510 50  0001 C CNN
+F 3 "~" V 1000 2510 50  0001 C CNN
+	1    1000 2450
 	1    0    0    -1
 $EndComp
@@
 L Regulator_Switching:LTC3525-5 U1
 U 1 1 613E4BD4
-P 2300 2300
-F 0 "U1" H 2400 2650 50  0000 C CNN
-F 1 "LTC3525-5" H 2550 2550 50  0000 C CNN
-F 2 "Package_TO_SOT_SMD:SOT-363_SC-70-6" H 2350 2050 50  0001 L CNN
-F 3 "https://www.analog.com/media/en/technical-documentation/data-sheets/3525fc.pdf" H 2300 2300 50  0001 C CNN
-	1    2300 2300
-	1    0    0    -1
-$EndComp
-Wire Wire Line
-	1800 2300 1900 2300
+P 2800 2300
+F 0 "U1" H 2900 2650 50  0000 C CNN
+F 1 "LTC3525-5" H 3050 2550 50  0000 C CNN
+F 2 "Package_TO_SOT_SMD:SOT-363_SC-70-6" H 2850 2050 50  0001 L CNN
+F 3 "https://www.analog.com/media/en/technical-documentation/data-sheets/3525fc.pdf" H 2800 2300 50  0001 C CNN
+	1    2800 2300
+	1    0    0    -1
+$EndComp
+Wire Wire Line
+	2300 2300 2400 2300
 $Comp
 L Device:L L1
 U 1 1 613E7FA8
-P 2600 1800
-F 0 "L1" V 2790 1800 50  0000 C CNN
-F 1 "10uH" V 2699 1800 50  0000 C CNN
-F 2 "Inductor_SMD:L_1210_3225Metric" H 2600 1800 50  0001 C CNN
-F 3 "~" H 2600 1800 50  0001 C CNN
-	1    2600 1800
+P 3100 1800
+F 0 "L1" V 3290 1800 50  0000 C CNN
+F 1 "10uH" V 3199 1800 50  0000 C CNN
+F 2 "Inductor_SMD:L_1210_3225Metric" H 3100 1800 50  0001 C CNN
+F 3 "~" H 3100 1800 50  0001 C CNN
+	1    3100 1800
 	0    -1   -1   0
 $EndComp
 Wire Wire Line
-	2850 1800 2850 2200
-Wire Wire Line
-	2850 2200 2700 2200
+	3350 1800 3350 2200
+Wire Wire Line
+	3350 2200 3200 2200
 $Comp
 L Device:C C2
 U 1 1 613EB1F1
-P 2900 2600
-F 0 "C2" H 3015 2646 50  0000 L CNN
-F 1 "10uF" H 3015 2555 50  0000 L CNN
-F 2 "Capacitor_SMD:C_0805_2012Metric" H 2938 2450 50  0001 C CNN
-F 3 "~" H 2900 2600 50  0001 C CNN
-	1    2900 2600
-	1    0    0    -1
-$EndComp
-Wire Wire Line
-	2900 2400 2900 2450
-Wire Wire Line
-	2700 2400 2900 2400
-Wire Wire Line
-	2900 2400 3000 2400
-Connection ~ 2900 2400
-Wire Wire Line
-	2300 2600 2300 2800
-Wire Wire Line
-	2300 2800 2900 2800
-Wire Wire Line
-	2900 2800 2900 2750
+P 3400 2600
+F 0 "C2" H 3515 2646 50  0000 L CNN
+F 1 "10uF" H 3515 2555 50  0000 L CNN
+F 2 "Capacitor_SMD:C_0805_2012Metric" H 3438 2450 50  0001 C CNN
+F 3 "~" H 3400 2600 50  0001 C CNN
+	1    3400 2600
+	1    0    0    -1
+$EndComp
+Wire Wire Line
+	3400 2400 3400 2450
+Wire Wire Line
+	3200 2400 3400 2400
+Wire Wire Line
+	3400 2400 3500 2400
+Connection ~ 3400 2400
+Wire Wire Line
+	2800 2600 2800 2800
+Wire Wire Line
+	2800 2800 3400 2800
+Wire Wire Line
+	3400 2800 3400 2750
 $Comp
 L Device:C C1
 U 1 1 613F1363
-P 1800 2600
-F 0 "C1" H 1915 2646 50  0000 L CNN
-F 1 "1uF" H 1915 2555 50  0000 L CNN
-F 2 "Capacitor_SMD:C_0805_2012Metric" H 1838 2450 50  0001 C CNN
-F 3 "~" H 1800 2600 50  0001 C CNN
-	1    1800 2600
-	1    0    0    -1
-$EndComp
-Wire Wire Line
-	2300 2800 1800 2800
-Wire Wire Line
-	1800 2800 1800 2750
-Connection ~ 2300 2800
-Wire Wire Line
-	1800 2450 1800 2300
-Wire Wire Line
-	2300 1800 2450 1800
-Wire Wire Line
-	2750 1800 2850 1800
-Wire Wire Line
-	1200 2600 1200 2800
-Wire Notes Line
-	1000 3150 3300 3150
-Wire Notes Line
-	3300 1500 1000 1500
+P 2300 2600
+F 0 "C1" H 2415 2646 50  0000 L CNN
+F 1 "1uF" H 2415 2555 50  0000 L CNN
+F 2 "Capacitor_SMD:C_0805_2012Metric" H 2338 2450 50  0001 C CNN
+F 3 "~" H 2300 2600 50  0001 C CNN
+	1    2300 2600
+	1    0    0    -1
+$EndComp
+Wire Wire Line
+	2800 2800 2300 2800
+Wire Wire Line
+	2300 2800 2300 2750
+Connection ~ 2800 2800
+Wire Wire Line
+	2300 2450 2300 2300
+Wire Wire Line
+	2800 1800 2950 1800
+Wire Wire Line
+	3250 1800 3350 1800
 $Comp
 L Light_trainer-rescue:+5V-power #PWR013
@@
 L Light_trainer-rescue:+5V-power #PWR08
 U 1 1 61414884
-P 3000 2350
-F 0 "#PWR08" H 3000 2200 50  0001 C CNN
-F 1 "+5V" H 3150 2400 50  0000 C CNN
-F 2 "" H 3000 2350 50  0001 C CNN
-F 3 "" H 3000 2350 50  0001 C CNN
-	1    3000 2350
-	1    0    0    -1
-$EndComp
-Wire Wire Line
-	3000 2350 3000 2400
+P 3500 2350
+F 0 "#PWR08" H 3500 2200 50  0001 C CNN
+F 1 "+5V" H 3650 2400 50  0000 C CNN
+F 2 "" H 3500 2350 50  0001 C CNN
+F 3 "" H 3500 2350 50  0001 C CNN
+	1    3500 2350
+	1    0    0    -1
+$EndComp
+Wire Wire Line
+	3500 2350 3500 2400
 $Comp
 L Light_trainer-rescue:GND-power #PWR05
 U 1 1 61415E58
-P 2300 2850
-F 0 "#PWR05" H 2300 2600 50  0001 C CNN
-F 1 "GND" H 2305 2677 50  0000 C CNN
-F 2 "" H 2300 2850 50  0001 C CNN
-F 3 "" H 2300 2850 50  0001 C CNN
-	1    2300 2850
-	1    0    0    -1
-$EndComp
-Wire Wire Line
-	2300 2850 2300 2800
-Wire Notes Line
-	3300 1500 3300 3150
-Wire Notes Line
-	1000 1500 1000 3150
+P 2800 2850
+F 0 "#PWR05" H 2800 2600 50  0001 C CNN
+F 1 "GND" H 2805 2677 50  0000 C CNN
+F 2 "" H 2800 2850 50  0001 C CNN
+F 3 "" H 2800 2850 50  0001 C CNN
+	1    2800 2850
+	1    0    0    -1
+$EndComp
+Wire Wire Line
+	2800 2850 2800 2800
+Wire Notes Line
+	3800 1500 3800 3150
+Wire Notes Line
+	800  1500 800  3150
 $Comp
 L Light_trainer-rescue:+5V-power #PWR017
@@
 L Connector:TestPoint TP2
 U 1 1 6143AF5D
-P 1800 1900
-F 0 "TP2" H 1858 2018 50  0000 L CNN
-F 1 "TestPoint" H 1858 1927 50  0000 L CNN
-F 2 "TestPoint:TestPoint_THTPad_2.5x2.5mm_Drill1.2mm" H 2000 1900 50  0001 C CNN
-F 3 "~" H 2000 1900 50  0001 C CNN
-F 4 "~" H 1800 1900 50  0001 C CNN "Fournisseur"
-F 5 "~" H 1800 1900 50  0001 C CNN "Prix total"
-F 6 "~" H 1800 1900 50  0001 C CNN "prix unité"
-	1    1800 1900
+P 2300 1900
+F 0 "TP2" H 2358 2018 50  0000 L CNN
+F 1 "TestPoint" H 2358 1927 50  0000 L CNN
+F 2 "TestPoint:TestPoint_THTPad_2.5x2.5mm_Drill1.2mm" H 2500 1900 50  0001 C CNN
+F 3 "~" H 2500 1900 50  0001 C CNN
+F 4 "~" H 2300 1900 50  0001 C CNN "Fournisseur"
+F 5 "~" H 2300 1900 50  0001 C CNN "Prix total"
+F 6 "~" H 2300 1900 50  0001 C CNN "prix unité"
+	1    2300 1900
 	1    0    0    -1
 $EndComp
@@
 L Connector:TestPoint TP3
 U 1 1 6143D663
-P 1800 2850
-F 0 "TP3" H 1600 3000 50  0000 L CNN
-F 1 "TestPoint" H 1400 2900 50  0000 L CNN
-F 2 "TestPoint:TestPoint_THTPad_2.5x2.5mm_Drill1.2mm" H 2000 2850 50  0001 C CNN
-F 3 "~" H 2000 2850 50  0001 C CNN
-F 4 "~" H 1800 2850 50  0001 C CNN "Fournisseur"
-F 5 "~" H 1800 2850 50  0001 C CNN "Prix total"
-F 6 "~" H 1800 2850 50  0001 C CNN "prix unité"
-	1    1800 2850
+P 2300 2850
+F 0 "TP3" H 2100 3000 50  0000 L CNN
+F 1 "TestPoint" H 1900 2900 50  0000 L CNN
+F 2 "TestPoint:TestPoint_THTPad_2.5x2.5mm_Drill1.2mm" H 2500 2850 50  0001 C CNN
+F 3 "~" H 2500 2850 50  0001 C CNN
+F 4 "~" H 2300 2850 50  0001 C CNN "Fournisseur"
+F 5 "~" H 2300 2850 50  0001 C CNN "Prix total"
+F 6 "~" H 2300 2850 50  0001 C CNN "prix unité"
+	1    2300 2850
 	-1   0    0    1
 $EndComp
 Wire Wire Line
-	1800 2800 1800 2850
+	2300 2800 2300 2850
 Wire Wire Line
 	6050 2950 6250 2950
@@
 Text Notes 4450 1450 0    50   ~ 0
 ESP DEVKIT C\n
-Text Notes 1000 1450 0    50   ~ 0
+Text Notes 1500 1450 0    50   ~ 0
 Alimentation 3 pile AA avec régulateur 5V\n
 Text Notes 4500 4550 0    50   ~ 0
@@
 L Device:Jumper JP1
 U 1 1 614DCE52
-P 1500 1950
-F 0 "JP1" H 1500 2214 50  0000 C CNN
-F 1 "Jumper" H 1500 2123 50  0000 C CNN
-F 2 "Jumper:SolderJumper-2_P1.3mm_Open_Pad1.0x1.5mm" H 1500 1950 50  0001 C CNN
-F 3 "~" H 1500 1950 50  0001 C CNN
-F 4 "~" H 1500 1950 50  0001 C CNN "Fournisseur"
-F 5 "~" H 1500 1950 50  0001 C CNN "Prix total"
-F 6 "~" H 1500 1950 50  0001 C CNN "prix unité"
-	1    1500 1950
-	1    0    0    -1
-$EndComp
-Wire Wire Line
-	2300 1800 2300 1950
-Wire Wire Line
-	1800 2300 1800 1950
-Connection ~ 1800 2300
-Wire Wire Line
-	1800 1950 1800 1900
-Connection ~ 1800 1950
-Wire Wire Line
-	1200 1950 1200 2200
-Wire Wire Line
-	1800 1950 2300 1950
+P 1900 1950
+F 0 "JP1" H 1900 2214 50  0000 C CNN
+F 1 "Jumper" H 1900 2123 50  0000 C CNN
+F 2 "Jumper:SolderJumper-2_P1.3mm_Open_Pad1.0x1.5mm" H 1900 1950 50  0001 C CNN
+F 3 "~" H 1900 1950 50  0001 C CNN
+F 4 "~" H 1900 1950 50  0001 C CNN "Fournisseur"
+F 5 "~" H 1900 1950 50  0001 C CNN "Prix total"
+F 6 "~" H 1900 1950 50  0001 C CNN "prix unité"
+	1    1900 1950
+	1    0    0    -1
+$EndComp
+Wire Wire Line
+	2800 1800 2800 1950
+Wire Wire Line
+	2300 2300 2300 1950
+Connection ~ 2300 2300
+Wire Wire Line
+	2300 1950 2300 1900
 Connection ~ 2300 1950
 Wire Wire Line
-	2300 1950 2300 2000
-Wire Wire Line
-	1200 2800 1800 2800
-Connection ~ 1800 2800
+	2300 1950 2800 1950
+Connection ~ 2800 1950
+Wire Wire Line
+	2800 1950 2800 2000
+Connection ~ 2300 2800
+$Comp
+L Switch:SW_SPDT SW5
+U 1 1 61410395
+P 1300 2050
+F 0 "SW5" H 1300 2335 50  0000 C CNN
+F 1 "SW_SPDT" H 1300 2244 50  0000 C CNN
+F 2 "Work_Forestier:C&K-1101M2S5CQE2" H 1300 2050 50  0001 C CNN
+F 3 "https://www.ckswitches.com/media/1429/1000.pdf" H 1300 2050 50  0001 C CNN
+	1    1300 2050
+	1    0    0    -1
+$EndComp
+Wire Wire Line
+	1000 2800 2300 2800
+Wire Wire Line
+	1000 2050 1100 2050
+NoConn ~ 1500 2150
+Wire Notes Line
+	800  1500 3800 1500
+Wire Notes Line
+	800  3150 3800 3150
+Wire Wire Line
+	2200 1950 2300 1950
+Wire Wire Line
+	1600 1950 1500 1950
+Wire Wire Line
+	1000 2650 1000 2800
+Wire Wire Line
+	1000 2250 1000 2050
 $EndSCHEMATC

Commit message: Creat Gerber
creation des fichiers gerber.
Parts:
- added H1, H2, H3, H4: MountingHole, MountingHole:MountingHole_3.2mm_M3, symbol Mechanical:MountingHole
- U2: symbol Work_Forestier:ESP32-DevKitC-32D -> Light_trainer-rescue:ESP32-DevKitC-32D-Work_Forestier
Other:
- note added: "Trous de fixation\n"
Changed lines of the file:
@@
 	1400 6750 1500 6750
 $Comp
-L Work_Forestier:ESP32-DevKitC-32D U2
+L Light_trainer-rescue:ESP32-DevKitC-32D-Work_Forestier U2
 U 1 1 6148669D
 P 5700 2900
@@
 Wire Wire Line
 	1000 2250 1000 2050
+$Comp
+L Mechanical:MountingHole H1
+U 1 1 6141B071
+P 7000 4750
+F 0 "H1" H 7100 4796 50  0000 L CNN
+F 1 "MountingHole" H 7100 4705 50  0000 L CNN
+F 2 "MountingHole:MountingHole_3.2mm_M3" H 7000 4750 50  0001 C CNN
+F 3 "~" H 7000 4750 50  0001 C CNN
+	1    7000 4750
+	1    0    0    -1
+$EndComp
+$Comp
+L Mechanical:MountingHole H2
+U 1 1 6141E6D1
+P 7800 4750
+F 0 "H2" H 7900 4796 50  0000 L CNN
+F 1 "MountingHole" H 7900 4705 50  0000 L CNN
+F 2 "MountingHole:MountingHole_3.2mm_M3" H 7800 4750 50  0001 C CNN
+F 3 "~" H 7800 4750 50  0001 C CNN
+	1    7800 4750
+	1    0    0    -1
+$EndComp
+$Comp
+L Mechanical:MountingHole H4
+U 1 1 6141E94E
+P 7800 5150
+F 0 "H4" H 7900 5196 50  0000 L CNN
+F 1 "MountingHole" H 7900 5105 50  0000 L CNN
+F 2 "MountingHole:MountingHole_3.2mm_M3" H 7800 5150 50  0001 C CNN
+F 3 "~" H 7800 5150 50  0001 C CNN
+	1    7800 5150
+	1    0    0    -1
+$EndComp
+$Comp
+L Mechanical:MountingHole H3
+U 1 1 6141EBEB
+P 7000 5150
+F 0 "H3" H 7100 5196 50  0000 L CNN
+F 1 "MountingHole" H 7100 5105 50  0000 L CNN
+F 2 "MountingHole:MountingHole_3.2mm_M3" H 7000 5150 50  0001 C CNN
+F 3 "~" H 7000 5150 50  0001 C CNN
+	1    7000 5150
+	1    0    0    -1
+$EndComp
+Wire Notes Line
+	6800 5400 8550 5400
+Wire Notes Line
+	8550 5400 8550 4550
+Wire Notes Line
+	8550 4550 6800 4550
+Wire Notes Line
+	6800 4550 6800 5400
+Text Notes 6800 4500 0    50   ~ 0
+Trous de fixation\n
 $EndSCHEMATC

Commit message: creat archive
creat archive V1
Parts:
- BT1: symbol Device:Battery -> archive:Device_Battery
- C1, C2: symbol Device:C -> archive:Device_C
- D1, D2, D3, D4, D5: symbol Light_trainer-rescue:SK6812-LED -> archive:Light_trainer-rescue_SK6812-LED
- H1, H2, H3, H4: symbol Mechanical:MountingHole -> archive:Mechanical_MountingHole
- JP1: symbol Device:Jumper -> archive:Device_Jumper
- L1: symbol Device:L -> archive:Device_L
- R1: symbol Light_trainer-rescue:R-Device -> archive:Light_trainer-rescue_R-Device
- SW1, SW2, SW3, SW4: symbol Light_trainer-rescue:SW_Push-Switch -> archive:Light_trainer-rescue_SW_Push-Switch
- SW5: symbol Switch:SW_SPDT -> archive:Switch_SW_SPDT
- TP1, TP4, TP5: symbol Light_trainer-rescue:TestPoint-Connector -> archive:Light_trainer-rescue_TestPoint-Connector
- TP2, TP3, TP6, TP7, TP8: symbol Connector:TestPoint -> archive:Connector_TestPoint
- U1: symbol Regulator_Switching:LTC3525-5 -> archive:Regulator_Switching_LTC3525-5
- U2: symbol Light_trainer-rescue:ESP32-DevKitC-32D-Work_Forestier -> archive:Light_trainer-rescue_ESP32-DevKitC-32D-Work_Forestier
Changed lines of the file:
@@
 $EndDescr
 $Comp
-L Light_trainer-rescue:SW_Push-Switch SW1
+L archive:Light_trainer-rescue_SW_Push-Switch SW1
 U 1 1 5FD2E185
 P 1600 4000
@@
 $EndComp
 $Comp
-L Light_trainer-rescue:SW_Push-Switch SW2
+L archive:Light_trainer-rescue_SW_Push-Switch SW2
 U 1 1 5FD62CD6
 P 1600 4350
@@
 $EndComp
 $Comp
-L Light_trainer-rescue:SW_Push-Switch SW3
+L archive:Light_trainer-rescue_SW_Push-Switch SW3
 U 1 1 5FD65B5A
 P 1600 4700
@@
 $EndComp
 $Comp
-L Light_trainer-rescue:SW_Push-Switch SW4
+L archive:Light_trainer-rescue_SW_Push-Switch SW4
 U 1 1 5FD68A79
 P 1600 5050
@@
 Connection ~ 1300 4700
 $Comp
-L Light_trainer-rescue:R-Device R1
+L archive:Light_trainer-rescue_R-Device R1
 U 1 1 5FD7C917
 P 1950 5300
@@
 	1950 5500 1950 5450
 $Comp
-L Light_trainer-rescue:+3.3V-power #PWR01
+L archive:Light_trainer-rescue_+3.3V-power #PWR01
 U 1 1 6047DC4D
 P 1300 3900
@@
 LightTrainer V00
 $Comp
-L Light_trainer-rescue:SK6812-LED D1
+L archive:Light_trainer-rescue_SK6812-LED D1
 U 1 1 5FDB63B9
 P 1800 6750
@@
 $EndComp
 $Comp
-L Light_trainer-rescue:SK6812-LED D2
+L archive:Light_trainer-rescue_SK6812-LED D2
 U 1 1 5FEF28E1
 P 2450 6750
@@
 $EndComp
 $Comp
-L Light_trainer-rescue:SK6812-LED D3
+L archive:Light_trainer-rescue_SK6812-LED D3
 U 1 1 5FF375C6
 P 3100 6750
@@
 $EndComp
 $Comp
-L Light_trainer-rescue:SK6812-LED D4
+L archive:Light_trainer-rescue_SK6812-LED D4
 U 1 1 5FF375CF
 P 3750 6750
@@
 LED néo-pixel
 $Comp
-L Light_trainer-rescue:GND-power #PWR014
+L archive:Light_trainer-rescue_GND-power #PWR014
 U 1 1 603F42F0
 P 4400 7100
@@
 $EndComp
 $Comp
-L Light_trainer-rescue:GND-power #PWR03
+L archive:Light_trainer-rescue_GND-power #PWR03
 U 1 1 6043A369
 P 1800 7100
@@
 $EndComp
 $Comp
-L Light_trainer-rescue:GND-power #PWR07
+L archive:Light_trainer-rescue_GND-power #PWR07
 U 1 1 6044BBB6
 P 2450 7100
@@
 $EndComp
 $Comp
-L Light_trainer-rescue:GND-power #PWR010
+L archive:Light_trainer-rescue_GND-power #PWR010
 U 1 1 6045D3E7
 P 3100 7100
@@
 $EndComp
 $Comp
-L Light_trainer-rescue:GND-power #PWR012
+L archive:Light_trainer-rescue_GND-power #PWR012
 U 1 1 6046ECE6
 P 3750 7100
@@
 $EndComp
 $Comp
-L Light_trainer-rescue:GND-power #PWR04
+L archive:Light_trainer-rescue_GND-power #PWR04
 U 1 1 60491CDF
 P 1950 5500
@@
 $EndComp
 $Comp
-L Light_trainer-rescue:+5V-power #PWR02
+L archive:Light_trainer-rescue_+5V-power #PWR02
 U 1 1 604E998D
 P 1800 6400
@@
 $EndComp
 $Comp
-L Light_trainer-rescue:+5V-power #PWR06
+L archive:Light_trainer-rescue_+5V-power #PWR06
 U 1 1 604FB129
 P 2450 6400
@@
 $EndComp
 $Comp
-L Light_trainer-rescue:+5V-power #PWR09
+L archive:Light_trainer-rescue_+5V-power #PWR09
 U 1 1 6050C9D7
 P 3100 6400
@@
 $EndComp
 $Comp
-L Light_trainer-rescue:+5V-power #PWR011
+L archive:Light_trainer-rescue_+5V-power #PWR011
 U 1 1 6051E1D9
 P 3750 6400
@@
 $EndComp
 $Comp
-L Light_trainer-rescue:TestPoint-Connector TP4
+L archive:Light_trainer-rescue_TestPoint-Connector TP4
 U 1 1 606B57C6
 P 1950 3850
@@
 	1950 3850 1950 4000
 $Comp
-L Light_trainer-rescue:TestPoint-Connector TP1
+L archive:Light_trainer-rescue_TestPoint-Connector TP1
 U 1 1 6070C247
 P 1400 6700
@@
 	1400 6750 1500 6750
 $Comp
-L Light_trainer-rescue:ESP32-DevKitC-32D-Work_Forestier U2
+L archive:Light_trainer-rescue_ESP32-DevKitC-32D-Work_Forestier U2
 U 1 1 6148669D
 P 5700 2900
@@
 $EndComp
 $Comp
-L Device:Battery BT1
+L archive:Device_Battery BT1
 U 1 1 613C716D
 P 1000 2450
@@
 $EndComp
 $Comp
-L Regulator_Switching:LTC3525-5 U1
+L archive:Regulator_Switching_LTC3525-5 U1
 U 1 1 613E4BD4
 P 2800 2300
@@
 	2300 2300 2400 2300
 $Comp
-L Device:L L1
+L archive:Device_L L1
 U 1 1 613E7FA8
 P 3100 1800
@@
 	3350 2200 3200 2200
 $Comp
-L Device:C C2
+L archive:Device_C C2
 U 1 1 613EB1F1
 P 3400 2600
@@
 	3400 2800 3400 2750
 $Comp
-L Device:C C1
+L archive:Device_C C1
 U 1 1 613F1363
 P 2300 2600
@@
 	3250 1800 3350 1800
 $Comp
-L Light_trainer-rescue:+5V-power #PWR013
+L archive:Light_trainer-rescue_+5V-power #PWR013
 U 1 1 60552CBF
 P 4400 6400
@@
 	4750 6700 4750 6750
 $Comp
-L Light_trainer-rescue:TestPoint-Connector TP5
+L archive:Light_trainer-rescue_TestPoint-Connector TP5
 U 1 1 60377721
 P 4750 6700
@@
 	4750 6750 4700 6750
 $Comp
-L Light_trainer-rescue:SK6812-LED D5
+L archive:Light_trainer-rescue_SK6812-LED D5
 U 1 1 5FF5112C
 P 4400 6750
@@
 $EndComp
 $Comp
-L Light_trainer-rescue:+5V-power #PWR08
+L archive:Light_trainer-rescue_+5V-power #PWR08
 U 1 1 61414884
 P 3500 2350
@@
 	3500 2350 3500 2400
 $Comp
-L Light_trainer-rescue:GND-power #PWR05
+L archive:Light_trainer-rescue_GND-power #PWR05
 U 1 1 61415E58
 P 2800 2850
@@
 	800  1500 800  3150
 $Comp
-L Light_trainer-rescue:+5V-power #PWR017
+L archive:Light_trainer-rescue_+5V-power #PWR017
 U 1 1 61421D85
 P 4900 3700
@@
 	5350 3750 4900 3750
 $Comp
-L Light_trainer-rescue:GND-power #PWR021
+L archive:Light_trainer-rescue_GND-power #PWR021
 U 1 1 61424DCF
 P 6350 2000
@@
 	6050 1950 6350 1950
 $Comp
-L Light_trainer-rescue:GND-power #PWR022
+L archive:Light_trainer-rescue_GND-power #PWR022
 U 1 1 61427B71
 P 6350 2600
@@
 	6050 2550 6350 2550
 $Comp
-L Light_trainer-rescue:GND-power #PWR016
+L archive:Light_trainer-rescue_GND-power #PWR016
 U 1 1 6142C078
 P 4900 3300
@@
 	5350 3250 4900 3250
 $Comp
-L Connector:TestPoint TP6
+L archive:Connector_TestPoint TP6
 U 1 1 6142F575
 P 4800 4850
@@
 $EndComp
 $Comp
-L Light_trainer-rescue:GND-power #PWR015
+L archive:Light_trainer-rescue_GND-power #PWR015
 U 1 1 61430156
 P 4800 4900
@@
 	4800 4900 4800 4850
 $Comp
-L Connector:TestPoint TP7
+L archive:Connector_TestPoint TP7
 U 1 1 61436086
 P 5350 4850
@@
 $EndComp
 $Comp
-L Light_trainer-rescue:+5V-power #PWR019
+L archive:Light_trainer-rescue_+5V-power #PWR019
 U 1 1 61439438
 P 5350 4950
@@
 	5350 4850 5350 4950
 $Comp
-L Connector:TestPoint TP2
+L archive:Connector_TestPoint TP2
 U 1 1 6143AF5D
 P 2300 1900
@@
 $EndComp
 $Comp
-L Connector:TestPoint TP3
+L archive:Connector_TestPoint TP3
 U 1 1 6143D663
 P 2300 2850
@@
 	5100 1850 5100 1950
 $Comp
-L Light_trainer-rescue:+3.3V-power #PWR018
+L archive:Light_trainer-rescue_+3.3V-power #PWR018
 U 1 1 6144B410
 P 5100 1850
@@
 Test point GND/5V\n
 $Comp
-L Connector:TestPoint TP8
+L archive:Connector_TestPoint TP8
 U 1 1 614C7562
 P 5900 4850
@@
 $EndComp
 $Comp
-L Light_trainer-rescue:+3.3V-power #PWR020
+L archive:Light_trainer-rescue_+3.3V-power #PWR020
 U 1 1 614C9C11
 P 5900 4950
@@
 	4500 5250 6400 5250
 $Comp
-L Device:Jumper JP1
+L archive:Device_Jumper JP1
 U 1 1 614DCE52
 P 1900 1950
@@
 Connection ~ 2300 2800
 $Comp
-L Switch:SW_SPDT SW5
+L archive:Switch_SW_SPDT SW5
 U 1 1 61410395
 P 1300 2050
@@
 	1000 2250 1000 2050
 $Comp
-L Mechanical:MountingHole H1
+L archive:Mechanical_MountingHole H1
 U 1 1 6141B071
 P 7000 4750
@@
 $EndComp
 $Comp
-L Mechanical:MountingHole H2
+L archive:Mechanical_MountingHole H2
 U 1 1 6141E6D1
 P 7800 4750
@@
 $EndComp
 $Comp
-L Mechanical:MountingHole H4
+L archive:Mechanical_MountingHole H4
 U 1 1 6141E94E
 P 7800 5150
@@
 $EndComp
 $Comp
-L Mechanical:MountingHole H3
+L archive:Mechanical_MountingHole H3
 U 1 1 6141EBEB
 P 7000 5150
