File: 4_Fabrication/Version_00/C_KiCAD/Light_trainer/Light_trainer.kicad_pcb (KiCad board)
At the start: 2 copper layers, 110 x 110 mm, 28 parts, among them SW1 SW_Push, SW2 SW_Push, SW3 SW_Push, SW4 SW_Push, SW5 SW_SPDT, U1 LTC3525-5, U2 ESP32-DevKitC-32D

Commit message: Creat Gerber
creation des fichiers gerber.
Parts:
- added H1: MountingHole, MountingHole:MountingHole_3.2mm_M3, F.Cu at (120.0, 140.0)
- added H2: MountingHole, MountingHole:MountingHole_3.2mm_M3, F.Cu at (160.0, 140.0)
- added H3: MountingHole, MountingHole:MountingHole_3.2mm_M3, F.Cu at (160.0, 60.0)
- added H4: MountingHole, MountingHole:MountingHole_3.2mm_M3, F.Cu at (120.0, 60.0)
- moved REF** 5.95 mm to (128.0, 67.0)
- moved REF** 5.68 mm to (118.0, 67.0)
Connections:
- SW5 pad 3: (no net) -> Net-(SW5-Pad3)
- U2 pad CLK: (no net) -> Net-(U2-PadCLK)
- U2 pad CMD: (no net) -> Net-(U2-PadCMD)
- U2 pad EN: (no net) -> Net-(U2-PadEN)
- U2 pad IO0: (no net) -> Net-(U2-PadIO0)
- U2 pad IO12: (no net) -> Net-(U2-PadIO12)
- U2 pad IO13: (no net) -> Net-(U2-PadIO13)
- U2 pad IO14: (no net) -> Net-(U2-PadIO14)
- U2 pad IO15: (no net) -> Net-(U2-PadIO15)
- U2 pad IO18: (no net) -> Net-(U2-PadIO18)
- U2 pad IO19: (no net) -> Net-(U2-PadIO19)
- U2 pad IO2: (no net) -> Net-(U2-PadIO2)
- U2 pad IO21: (no net) -> Net-(U2-PadIO21)
- U2 pad IO22: (no net) -> Net-(U2-PadIO22)
- U2 pad IO23: (no net) -> Net-(U2-PadIO23)
- U2 pad IO25: (no net) -> Net-(U2-PadIO25)
- U2 pad IO26: (no net) -> Net-(U2-PadIO26)
- U2 pad IO27: (no net) -> Net-(U2-PadIO27)
- U2 pad IO32: (no net) -> Net-(U2-PadIO32)
- U2 pad IO33: (no net) -> Net-(U2-PadIO33)
- U2 pad IO34: (no net) -> Net-(U2-PadIO34)
- U2 pad IO35: (no net) -> Net-(U2-PadIO35)
- U2 pad IO4: (no net) -> Net-(U2-PadIO4)
- U2 pad IO5: (no net) -> Net-(U2-PadIO5)
- U2 pad RXD0: (no net) -> Net-(U2-PadRXD0)
- U2 pad SD0: (no net) -> Net-(U2-PadSD0)
- U2 pad SD1: (no net) -> Net-(U2-PadSD1)
- U2 pad SD2: (no net) -> Net-(U2-PadSD2)
- U2 pad SD3: (no net) -> Net-(U2-PadSD3)
- U2 pad SVN: (no net) -> Net-(U2-PadSVN)
- U2 pad SVP: (no net) -> Net-(U2-PadSVP)
- U2 pad TXD0: (no net) -> Net-(U2-PadTXD0)
Routing:
- net +3V3: track 266.0 -> 268.8 mm
- net +5V: track 285.3 -> 286.5 mm
- net GND: track 277.3 -> 278.4 mm, vias 136 -> 137
- net switch: track 259.9 -> 258.9 mm
Other:
- rule pad_to_mask_clearance: 0.05 -> 0

Commit message: add pdf fabrication
add pdf fabrication
Other:
- board text added: "BOT LAYER"
- board text added: "BOT SILKSCREEN"
- board text added: "BOT SOLDERMASK"
- board text added: "EDGE CUT"
- board text added: "TOP LAYER"
- board text added: "TOP PASTE"
- board text added: "TOP SILKSCREEN"
- board text added: "TOP SOLDERMASK"
